File: kicad/nwX287.kicad_sch (KiCad schematic)
At the start: 4 parts, among them U1 bq3285, U2 Socket, Y1 32.768kHz 6pF

Commit message: adjust layout and silkscreen
Other:
- moved on the sheet: BT1, Y1
Changed lines of the file:
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@@
 	(global_label "GND"
 		(shape input)
-		(at 121.92 41.91 180)
-		(effects
-			(font
-				(size 1.27 1.27)
-			)
-			(justify right)
-		)
-		(property "Intersheetrefs" "${INTERSHEET_REFS}"
-			(at 121.92 41.91 0)
+		(at 92.71 40.64 180)
+		(effects
+			(font
+				(size 1.27 1.27)
+			)
+			(justify right)
+		)
+		(property "Intersheetrefs" "${INTERSHEET_REFS}"
+			(at 92.71 40.64 0)
 			(hide yes)
 			(show_name no)
@@
 	(global_label "X1"
 		(shape input)
-		(at 127 45.72 270)
-		(effects
-			(font
-				(size 1.27 1.27)
-			)
-			(justify right)
-		)
-		(property "Intersheetrefs" "${INTERSHEET_REFS}"
-			(at 127 45.72 0)
+		(at 97.79 44.45 270)
+		(effects
+			(font
+				(size 1.27 1.27)
+			)
+			(justify right)
+		)
+		(property "Intersheetrefs" "${INTERSHEET_REFS}"
+			(at 97.79 44.45 0)
 			(hide yes)
 			(show_name no)
@@
 	(global_label "GND"
 		(shape input)
-		(at 161.29 45.72 270)
-		(effects
-			(font
-				(size 1.27 1.27)
-			)
-			(justify right)
-		)
-		(property "Intersheetrefs" "${INTERSHEET_REFS}"
-			(at 161.29 45.72 0)
+		(at 135.89 44.45 270)
+		(effects
+			(font
+				(size 1.27 1.27)
+			)
+			(justify right)
+		)
+		(property "Intersheetrefs" "${INTERSHEET_REFS}"
+			(at 135.89 44.45 0)
 			(hide yes)
 			(show_name no)
@@
 	(global_label "X2"
 		(shape input)
-		(at 127 38.1 90)
+		(at 97.79 36.83 90)
 		(effects
 			(font
@@
 		)
 		(property "Intersheetrefs" "${INTERSHEET_REFS}"
-			(at 127 38.1 0)
+			(at 97.79 36.83 0)
 			(hide yes)
 			(show_name no)
@@
 	(global_label "BC"
 		(shape input)
-		(at 161.29 38.1 90)
+		(at 135.89 36.83 90)
 		(effects
 			(font
@@
 		)
 		(property "Intersheetrefs" "${INTERSHEET_REFS}"
-			(at 161.29 38.1 0)
+			(at 135.89 36.83 0)
 			(hide yes)
 			(show_name no)
@@
 	(symbol
 		(lib_id "Device:Crystal_GND3")
-		(at 127 41.91 270)
+		(at 97.79 40.64 270)
 		(unit 1)
 		(body_style 1)
@@
 		(dnp no)
 		(property "Reference" "Y1"
-			(at 132.08 40.64 90)
+			(at 102.87 39.37 90)
 			(show_name no)
 			(do_not_autoplace no)
@@
 		)
 		(property "Value" "32.768kHz 6pF"
-			(at 137.16 43.18 90)
+			(at 107.95 41.91 90)
 			(show_name no)
 			(do_not_autoplace no)
@@
 		)
 		(property "Footprint" "Crystal:Crystal_SMD_FrontierElectronics_FM206"
-			(at 127 41.91 0)
+			(at 97.79 40.64 0)
 			(hide yes)
 			(show_name no)
@@
 		)
 		(property "Datasheet" "~"
-			(at 127 41.91 0)
+			(at 97.79 40.64 0)
 			(hide yes)
 			(show_name no)
@@
 		)
 		(property "Description" "Three pin crystal, GND on pin 3"
-			(at 127 30.988 90)
+			(at 97.79 29.718 90)
 			(show_name no)
 			(do_not_autoplace no)
@@
 	(symbol
 		(lib_id "Device:Battery_Cell")
-		(at 161.29 43.18 0)
+		(at 135.89 41.91 0)
 		(unit 1)
 		(body_style 1)
@@
 		(dnp no)
 		(property "Reference" "BT1"
-			(at 164.2872 40.7416 0)
+			(at 138.8872 39.4716 0)
 			(show_name no)
 			(do_not_autoplace no)
@@
 		)
 		(property "Value" "CR2032"
-			(at 164.2872 43.053 0)
+			(at 138.8872 41.783 0)
 			(show_name no)
 			(do_not_autoplace no)
@@
 		)
 		(property "Footprint" "Battery:BatteryHolder_MYOUNG_BS-07-A1BJ001_CR2032"
-			(at 161.29 41.656 90)
+			(at 135.89 40.386 90)
 			(hide yes)
 			(show_name no)
@@
 		)
 		(property "Datasheet" "~"
-			(at 161.29 41.656 90)
+			(at 135.89 40.386 90)
 			(hide yes)
 			(show_name no)
@@
 		)
 		(property "Description" "Single-cell battery"
-			(at 161.29 30.988 0)
+			(at 135.89 29.718 0)
 			(show_name no)
 			(do_not_autoplace no)
@@
 		)
 		(property "Sim.Device" "V"
-			(at 161.29 43.18 0)
+			(at 135.89 41.91 0)
 			(hide yes)
 			(show_name no)
@@
 		)
 		(property "Sim.Type" "DC"
-			(at 161.29 43.18 0)
+			(at 135.89 41.91 0)
 			(hide yes)
 			(show_name no)
@@
 		)
 		(property "Sim.Pins" "1=+ 2=-"
-			(at 161.29 43.18 0)
-			(hide yes)
-			(show_name no)
+			(at 135.89 41.91 0)
+			(hide yes)
+			(show_name no)
