File: pcb/rtc.kicad_pcb (KiCad board)
At the start: 2 copper layers, 52.5 x 24 mm, 4 parts, among them U1 bq3285, U2 Socket, Y1 32.768kHz 6pF

Commit message: various changes
Other:
- board text added: "CTRNNR RTC INT CR2032"
- board text added: "github.com/CityRunner/rtc-int-cr2032"
- board text removed: "CTRNNR INT RTC CR2032"
- board text removed: "github.com/CityRunner/rtc-cr2032-ssop"

Commit message: update pcb
Routing:
- net X1: track 6.37 -> 7.91 mm
- net SQW: track 14.0 -> 13.3 mm
Other:
- board text added: "VCC SQW NC RC NC INT RST DS NC RW AS CS"
- board text removed: "VCC SQW NC RCL NC INT RST DS NC R/W AS CS"
